File: PCBs/Thumb Cluster/crosses-wired-thumb-cluster.kicad_sch (KiCad schematic)
At the start: 44 parts, among them J1 Conn_01x03, J2 USB_C_Receptacle_USB2.0_16P, J3 Conn_01x14_Pin, J4 AudioJack4, SW1 SW_Push, SW2 SW_Push, SW3 SW_Push, SW4 SW_Push, U1 RP2040, U2 W25Q128JVS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

Commit message: Finished routing right side thumb cluster
Parts:
- C2, C3: footprint Capacitor_SMD:C_0402_1005Metric -> Capacitor_SMD:C_0603_1608Metric
Connections:
- net R-COL0: now also U1.14 (GPIO11)
- net R-COL1: now also U1.15 (GPIO12)
- net R-COL2: now also U1.18 (GPIO15)
- net R-COL3: now also U1.17 (GPIO14)
- net R-COL4: now also U1.16 (GPIO13)
- net R-COLP: now also U1.29 (GPIO18)
- net R-ROW0: now also U1.13 (GPIO10)
- net R-ROW1: now also U1.12 (GPIO9)
- net R-ROW2: now also U1.28 (GPIO17)
- net R-ROW3: now also U1.31 (GPIO20)
- net R-ROWH: now also U1.30 (GPIO19)
- net R-SERIAL: now also U1.41 (GPIO29/ADC3)
- net R-USB_DN: now also R2.2, U1.46 (USB_DM)
- net R-USB_DP: now also R3.1, U1.47 (USB_DP)
- no-connect marks 6 -> 7
Other:
- moved on the sheet: R2, R3
